File: kicad/cpu/tester/io-breakout.kicad_pcb (KiCad board)
At the start: 2 copper layers, 3 parts

Commit message: Wired
Parts:
- removed REF** (x2): PinHeader_1x28_P2.54mm_Vertical, Connector_PinHeader_2.54mm:PinHeader_1x28_P2.54mm_Vertical
- removed REF**: TSSOP-56_6.1x14mm_P0.5mm, Package_SO:TSSOP-56_6.1x14mm_P0.5mm
- added J1: Conn_01x28_Male, Connector_PinHeader_2.54mm:PinHeader_1x28_P2.54mm_Vertical, B.Cu at (104.1, 68.6)
- added J2: Conn_01x28_Male, Connector_PinHeader_2.54mm:PinHeader_1x28_P2.54mm_Vertical, B.Cu at (172.7, 53.3)
- added U1: PCA9698, Package_SO:TSSOP-56_6.1x14mm_P0.5mm, F.Cu at (138.4, 61.0)
Routing:
- net Net-(J1-Pad1): track 0.00 -> 29.7 mm
- net Net-(J2-Pad28): track 0.00 -> 29.7 mm
- net Net-(J1-Pad28): track 0.00 -> 29.7 mm
- net Net-(J2-Pad1): track 0.00 -> 29.7 mm
- net (no net): track 28.7 -> 0.00 mm
- net Net-(J1-Pad27): track 0.00 -> 27.5 mm
- net Net-(J1-Pad2): track 0.00 -> 27.5 mm
- net Net-(J2-Pad2): track 0.00 -> 27.5 mm
- net Net-(J2-Pad27): track 0.00 -> 27.5 mm
- net Net-(J2-Pad26): track 0.00 -> 26.4 mm, vias 0 -> 1
- net Net-(J1-Pad3): track 0.00 -> 26.4 mm, vias 0 -> 1
- net Net-(J2-Pad3): track 0.00 -> 26.4 mm, vias 0 -> 1
- net Net-(J1-Pad26): track 0.00 -> 26.4 mm, vias 0 -> 1
- net Net-(J2-Pad25): track 0.00 -> 25.0 mm, vias 0 -> 1
- net Net-(J1-Pad4): track 0.00 -> 25.0 mm, vias 0 -> 1
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Other:
- board outline added: 73.7 x 20.3 mm
- net class Default: clearance 0.2 -> 0.15; trace_width 0.25 -> 0.15
- rule trace_clearance: 0.2 -> 0.15
- rule trace_min: 0.2 -> 0.15

Commit message: Add plot files
Other:
- board text added: "Rhobotify Ltd"
- board text added: "io-breakout_1.0"
